Commit message: Launch files modified

File: urdf/hand_reflex.xacro (robot description, xacro)
@@ -480,4 +480,5 @@
       <joint name="finger_1_1_to_finger_1_2">
           <hardwareInterface>hardware_interface/EffortJointInterface</hardwareInterface>
+      </joint>
   </transmission>
   <transmission name="finger1_3_trans" type="SimpleTransmission">
@@ -488,4 +489,5 @@
       <joint name="finger_1_2_to_finger_1_3">
           <hardwareInterface>hardware_interface/EffortJointInterface</hardwareInterface>
+      </joint>
   </transmission>
   <transmission name="finger2_1_trans" type="SimpleTransmission">
@@ -505,4 +507,5 @@
       <joint name="finger_2_1_to_finger_2_2">
           <hardwareInterface>hardware_interface/EffortJointInterface</hardwareInterface>
+      </joint>
   </transmission>
   <transmission name="finger2_3_trans" type="SimpleTransmission">
@@ -513,4 +516,5 @@
       <joint name="finger_2_2_to_finger_2_3">
           <hardwareInterface>hardware_interface/EffortJointInterface</hardwareInterface>
+      </joint>
   </transmission>
   <transmission name="finger2_3_trans" type="SimpleTransmission">
@@ -521,4 +525,5 @@
       <joint name="base_to_finger_3_2">
           <hardwareInterface>hardware_interface/EffortJointInterface</hardwareInterface>
+      </joint>
   </transmission>
   <transmission name="finger3_3_trans" type="SimpleTransmission">
