Commit message: Screwdriver scenario with holes

File: urdf/object.urdf (robot description, URDF)
Before this commit: robot cyl, 1 links, 0 joints
Links:
- link cyl_object: geometry collision mesh filename=package://hand_simulator/meshes/screwdriver.STL; visual mesh filename=package://hand_simulator/meshes/screwdriver.STL
