Commit message: Rounded distals in T42

File: urdf/hand_T42.xacro (robot description, xacro)
@@ -128,13 +128,15 @@
                 <color rgba="0.1 1.0 0.1 1.0" />
             </material>
-            <origin xyz="-0.015875 -0.011709 -0.048006" />
-            <geometry>
-                <mesh filename="package://hand_simulator/meshes/distal_t42.STL" scale="0.025400 0.025400 0.025400" />
+            <origin xyz="-0.0 -0.0 -0.0" />
+            <!-- <origin xyz="-0.015875 -0.011709 -0.048006" /> -->  <!-- Pointed distal tips -->
+            <geometry>
+                <mesh filename="package://hand_simulator/meshes/distal_round_t42.STL" scale="0.001 0.001 0.001" />
+                <!-- <mesh filename="package://hand_simulator/meshes/distal_t42.STL" scale="0.025400 0.025400 0.025400" /> --> <!-- Pointed distal tips -->
             </geometry>
         </visual>
         <collision>
-            <origin xyz="-0.015875 -0.011709 -0.048006" />
-            <geometry>
-                <mesh filename="package://hand_simulator/meshes/distal_t42.STL" scale="0.025400 0.025400 0.025400" />
+            <origin xyz="-0.0 -0.0 -0.0" />
+            <geometry>
+                <mesh filename="package://hand_simulator/meshes/distal_round_t42.STL" scale="0.001 0.001 0.001" />
             </geometry>
         </collision>
@@ -198,13 +200,13 @@
                 <color rgba="0.9 0.3 0.1 1.0" />
             </material>
-            <origin xyz="-0.015875 -0.011709 -0.048006" />
-            <geometry>
-                <mesh filename="package://hand_simulator/meshes/distal_t42.STL" scale="0.025400 0.025400 0.025400" />
+            <origin xyz="0 0 0" />
+            <geometry>
+                <mesh filename="package://hand_simulator/meshes/distal_round_t42.STL" scale="0.001 0.001 0.001" />
             </geometry>
         </visual>
         <collision>
-            <origin xyz="-0.015875 -0.011709 -0.048006" />
-            <geometry>
-                <mesh filename="package://hand_simulator/meshes/distal_t42.STL" scale="0.025400 0.025400 0.025400" />
+            <origin xyz="0 0 0" />
+            <geometry>
+                <mesh filename="package://hand_simulator/meshes/distal_round_t42.STL" scale="0.001 0.001 0.001" />
             </geometry>
         </collision>

Commit message: Tuned for RL

File: urdf/hand_T42.xacro (robot description, xacro)
@@ -19,5 +19,5 @@
     <color rgba="0.106 0.227 0.631 1"/>
   </xacro:macro>
-  <xacro:property name="rubber_friction_coefficient" value="1.16" />
+  <xacro:property name="rubber_friction_coefficient" value="1.16" />  <!-- True: 1.16 -->
   <xacro:property name="rubber_contact_stiffness_coefficient" value="1000000.0" />
   <xacro:property name="rubber_contact_damping_coefficient" value="1.0" />
@@ -95,5 +95,5 @@
         <inertial>
             <origin xyz="-0.015875 -0.009000 -0.071550" />
-            <mass value="0.1" />
+            <mass value="0.1" />  <!-- 0.018485 -->
             <inertia ixx="0.01" ixy="0.0" ixz="0.0" iyy="0.01" iyz="0.0" izz="0.01" />
         </inertial>
@@ -121,5 +121,5 @@
         <inertial>
             <origin xyz="-0.015875 -0.011709 -0.048006" />
-            <mass value="0.1" />
+            <mass value="0.1" /> <!-- 0.02369 -->
             <inertia ixx="0.01" ixy="0.0" ixz="0.0" iyy="0.01" iyz="0.0" izz="0.01" />
         </inertial>

File: urdf/object.urdf (robot description, URDF)
Before this commit: robot cyl, 1 links, 0 joints
Links:
- link cyl_object: geometry collision cylinder length=0.09 radius=0.018; visual cylinder length=0.09 radius=0.018

Commit message: Added joint velocities feedback and joint damping within code

File: urdf/hand_T42.xacro (robot description, xacro)
@@ -23,4 +23,6 @@
   <xacro:property name="rubber_contact_damping_coefficient" value="1.0" />
   <xacro:property name="swivel_distance" value="0.0260" /> <!-- Not sure if this is the right distance for T42 -->
+  <xacro:property name="joint_damping_coefficient" value="5.0" />
+  <xacro:property name="joint_friction_coefficient" value="0.0" />
   <link name="world" />
     <link name="rail">
@@ -115,5 +117,5 @@
     </link>
     <gazebo reference="finger_1_1">
-      <selfCollide>true</selfCollide>
+      <selfCollide>false</selfCollide>
       <material>Gazebo/Red</material>
     </gazebo>
@@ -143,5 +145,5 @@
     </link>
     <gazebo reference="finger_1_2">
-      <selfCollide>true</selfCollide>
+      <selfCollide>false</selfCollide>
       <mu1>${rubber_friction_coefficient}</mu1>
       <mu2>${rubber_friction_coefficient}</mu2>
@@ -187,5 +189,5 @@
     </link>
     <gazebo reference="finger_2_1">
-      <selfCollide>true</selfCollide>
+      <selfCollide>false</selfCollide>
       <material>Gazebo/Red</material>
     </gazebo>
@@ -213,5 +215,5 @@
     </link>
     <gazebo reference="finger_2_2">
-      <selfCollide>true</selfCollide>
+      <selfCollide>false</selfCollide>
       <mu1>${rubber_friction_coefficient}</mu1>
       <mu2>${rubber_friction_coefficient}</mu2>
@@ -306,5 +308,5 @@
         <limit effort="10000" lower="0.0" upper="3.0" velocity="2" />
         <axis xyz="1 0 0" />
-        <dynamics damping="5" friction="0.0" />
+        <dynamics damping="${joint_damping_coefficient}" friction="${joint_friction_coefficient}" />
     </joint>
     <joint name="finger_1_1_to_finger_1_2" type="revolute">
@@ -314,5 +316,5 @@
         <limit effort="10000" lower="0.0" upper="1.57" velocity="2" />
         <axis xyz="1 0 0" />
-        <dynamics damping="5" friction="0.0" />
+        <dynamics damping="${joint_damping_coefficient}" friction="${joint_friction_coefficient}" />
     </joint>
     <joint name="base_link_to_swivel_2" type="fixed">
@@ -327,5 +329,5 @@
         <limit effort="10000" lower="0.0" upper="3.0" velocity="2" />
         <axis xyz="1 0 0" />
-        <dynamics damping="5" friction="0.0" />
+        <dynamics damping="${joint_damping_coefficient}" friction="${joint_friction_coefficient}" />
     </joint>
     <joint name="finger_2_1_to_finger_2_2" type="revolute">
@@ -335,5 +337,5 @@
         <limit effort="10000" lower="0.0" upper="1.57" velocity="2" />
         <axis xyz="1 0 0" />
-        <dynamics damping="5" friction="0.0" />
+        <dynamics damping="${joint_damping_coefficient}" friction="${joint_friction_coefficient}" />
     </joint>
  <!-- Transmissions -->

Commit message: Added damping and object velocity topic

File: urdf/hand_T42.xacro (robot description, xacro)
@@ -23,6 +23,6 @@
   <xacro:property name="rubber_contact_damping_coefficient" value="1.0" />
   <xacro:property name="swivel_distance" value="0.0260" /> <!-- Not sure if this is the right distance for T42 -->
-  <xacro:property name="joint_damping_coefficient" value="5.0" />
-  <xacro:property name="joint_friction_coefficient" value="0.0" />
+  <xacro:property name="joint_damping_coefficient" value="7.0" />
+  <xacro:property name="joint_friction_coefficient" value="0.4" />
   <link name="world" />
     <link name="rail">

Commit message: Added custom damping and velocity filters

File: urdf/hand_T42.xacro (robot description, xacro)
@@ -24,5 +24,5 @@
   <xacro:property name="swivel_distance" value="0.0260" /> <!-- Not sure if this is the right distance for T42 -->
   <xacro:property name="joint_damping_coefficient" value="7.0" />
-  <xacro:property name="joint_friction_coefficient" value="0.4" />
+  <xacro:property name="joint_friction_coefficient" value="0.0" />
   <link name="world" />
     <link name="rail">

Commit message: Screwdriver fix

File: urdf/hand_T42.xacro (robot description, xacro)
@@ -295,5 +295,5 @@
         <child link="base_link" />
         <axis xyz="0 0 1"/>
-        <limit effort="1000.0" lower="-100." upper="100." velocity="1"/>
+        <limit effort="1000.0" lower="-100." upper="100." velocity="0.25"/>
     </joint>
     <joint name="base_link_to_swivel_1" type="fixed">
