Commit message: Filled finger

File: urdf/hand_T42b.xacro (robot description, xacro)
@@ -131,8 +131,8 @@
                 <color rgba="0.1 1.0 0.1 1.0" />
             </material>
-            <origin xyz="-0.0 -0.0 -0.0" />
-            <!-- <origin xyz="-0.015875 -0.011709 -0.048006" /> -->  <!-- Pointed distal tips -->
-            <geometry>
-                <mesh filename="package://hand_simulator/meshes/distal_round_t42.STL" scale="0.001 0.001 0.001" />
+            <!-- <origin xyz="-0.0 -0.0 -0.0" /> -->
+            <origin xyz="-0.015875 -0.011709 -0.048006" />  <!-- Pointed distal tips -->
+            <geometry>
+                <mesh filename="package://hand_simulator/meshes/distal_round_t42_filled.STL" scale="0.001 0.001 0.001" />
                 <!-- <mesh filename="package://hand_simulator/meshes/distal_t42.STL" scale="0.025400 0.025400 0.025400" /> --> <!-- Pointed distal tips -->
             </geometry>
@@ -141,5 +141,5 @@
             <origin xyz="-0.0 -0.0 -0.0" />
             <geometry>
-                <mesh filename="package://hand_simulator/meshes/distal_round_t42.STL" scale="0.001 0.001 0.001" />
+                <mesh filename="package://hand_simulator/meshes/distal_round_t42_filled.STL" scale="0.001 0.001 0.001" />
             </geometry>
         </collision>
@@ -203,7 +203,7 @@
                 <color rgba="0.9 0.3 0.1 1.0" />
             </material>
-            <origin xyz="0 0 0" />
-            <geometry>
-                <mesh filename="package://hand_simulator/meshes/distal_round_t42.STL" scale="0.001 0.001 0.001" />
+            <origin xyz="-0.015875 -0.011709 -0.048006" />
+            <geometry>
+                <mesh filename="package://hand_simulator/meshes/distal_round_t42_filled.STL" scale="0.001 0.001 0.001" />
             </geometry>
         </visual>
@@ -211,5 +211,5 @@
             <origin xyz="0 0 0" />
             <geometry>
-                <mesh filename="package://hand_simulator/meshes/distal_round_t42.STL" scale="0.001 0.001 0.001" />
+                <mesh filename="package://hand_simulator/meshes/distal_round_t42_filled.STL" scale="0.001 0.001 0.001" />
             </geometry>
         </collision>
@@ -292,5 +292,5 @@
     </joint>
     <joint name="rail_to_base" type="prismatic">
-        <origin rpy="0 0 0" xyz="-0. 0.0 0.2" />
+        <origin rpy="0 0 0" xyz="-0. 0.0 0.3" />
         <parent link="rail" />
         <child link="base_link" />
@@ -312,5 +312,5 @@
     </joint>
     <joint name="finger_1_1_to_finger_1_2" type="revolute">
-        <origin rpy="0 0 0" xyz="0.000000 0.000000 -0.062551" />
+        <origin rpy="0 0 0" xyz="-0.0 -0.0 -0.062551" />
         <parent link="finger_1_1" />
         <child link="finger_1_2" />
@@ -333,5 +333,6 @@
     </joint>
     <joint name="finger_2_1_to_finger_2_2" type="revolute">
-        <origin rpy="0 0 0" xyz="0.000000 0.000000 -0.062551" />
+        <!-- <origin rpy="0 0 0" xyz="-0.01580000 -0.011800 -0.1105" /> -->
+        <origin rpy="0 0 0" xyz="-0.0 -0.0 -0.062551" />
         <parent link="finger_2_1" />
         <child link="finger_2_2" />
